File: watson-assistant.sch (KiCad schematic (older format))
At the start: 44 parts, among them J3 40HAT, J6 CONN_02X02, J9 CONN_01X02, Q1 DMG2305UX, Q2 DMMT5401, Q3 ELECTRET, U1 WM8731, U2 CAT24C32, U3 SN74AHCT125

Commit message: First version with all pcb nets connected
Connections:
- net P3V3 is gone; now on net +3V3: J6.1 (P1), R29.1, R6.1, R7.2, R8.1, U2.8 (VCC)
- net P5V is gone; now on net +5V: J6.3 (P3), Q1.3 (D), Q2.6 (E), R9.2
- net +3V3: no longer J3.1 (P3V3), J6.2 (P2), R7.1
- net +5V: no longer J3.2 (P5V), J3.4 (P5V), J6.4 (P4), Q1.2 (S), Q2.5 (E), R9.1
- new net P3V3_HAT: J3.1 (P3V3), J6.2 (P2), R7.1
- new net P5V_HAT: J3.2 (P5V), J3.4 (P5V), J6.4 (P4), Q1.2 (S), Q2.5 (E), R9.1
Changed lines of the file:
@@
 P5V
 Wire Wire Line
-	5250 4600 5850 4600
-Wire Wire Line
-	5250 4700 5850 4700
+	5200 4600 5850 4600
+Wire Wire Line
+	4850 4700 5850 4700
 Text Label 6950 4600 2    60   ~ 0
 P3V3_HAT
@@
 L +3.3V #PWR011
 U 1 1 59923D66
-P 7700 2400
-F 0 "#PWR011" H 7700 2250 50  0001 C CNN
-F 1 "+3.3V" H 7700 2540 50  0000 C CNN
-F 2 "" H 7700 2400 50  0001 C CNN
-F 3 "" H 7700 2400 50  0001 C CNN
-	1    7700 2400
+P 5200 4500
+F 0 "#PWR011" H 5200 4350 50  0001 C CNN
+F 1 "+3.3V" H 5200 4640 50  0000 C CNN
+F 2 "" H 5200 4500 50  0001 C CNN
+F 3 "" H 5200 4500 50  0001 C CNN
+	1    5200 4500
 	1    0    0    -1
 $EndComp
@@
 Text Label 3750 3050 0    60   ~ 0
 GPIO18
-Wire Wire Line
-	7700 2400 8150 2400
-Text Label 8150 2400 0    60   ~ 0
-P3V3_HAT
 $Comp
 L +5V #PWR027
 U 1 1 59928CE4
-P 7200 2350
-F 0 "#PWR027" H 7200 2200 50  0001 C CNN
-F 1 "+5V" H 7200 2490 50  0000 C CNN
-F 2 "" H 7200 2350 50  0001 C CNN
-F 3 "" H 7200 2350 50  0001 C CNN
-	1    7200 2350
+P 4850 4600
+F 0 "#PWR027" H 4850 4450 50  0001 C CNN
+F 1 "+5V" H 4850 4740 50  0000 C CNN
+F 2 "" H 4850 4600 50  0001 C CNN
+F 3 "" H 4850 4600 50  0001 C CNN
+	1    4850 4600
 	1    0    0    -1
 $EndComp
@@
 Wire Wire Line
 	10750 5400 10750 5350
+Wire Wire Line
+	4850 4600 4850 4700
+Wire Wire Line
+	5200 4500 5200 4600
 $EndSCHEMATC

Commit message: Add terminal for speaker output
This adds a terminal for a speaker. None of the commonly available pcb
mount speakers fit on the hat board with all the other components, so
this adds a terminal on the left edge to wire a speaker to.
Parts:
- added LS1: Speaker, Connectors_Terminal_Blocks:TerminalBlock_Pheonix_PT-3.5mm_2pol, symbol Speaker
Connections:
- net GND: now also LS1.2
- net L_OUT: now also LS1.1
Changed lines of the file:
@@
 A_VDD
 $Comp
-L +5V #PWR?
+L +5V #PWR030
 U 1 1 5993C6ED
 P 10750 5350
-F 0 "#PWR?" H 10750 5200 50  0001 C CNN
+F 0 "#PWR030" H 10750 5200 50  0001 C CNN
 F 1 "+5V" H 10750 5490 50  0000 C CNN
 F 2 "" H 10750 5350 50  0000 C CNN
@@
 Wire Wire Line
 	5200 4500 5200 4600
+$Comp
+L Speaker LS1
+U 1 1 5993D38A
+P 3500 9450
+F 0 "LS1" H 3550 9675 50  0000 R CNN
+F 1 "Speaker" H 3550 9600 50  0000 R CNN
+F 2 "Connectors_Terminal_Blocks:TerminalBlock_Pheonix_PT-3.5mm_2pol" H 3500 9250 50  0001 C CNN
+F 3 "" H 3490 9400 50  0001 C CNN
+	1    3500 9450
+	1    0    0    -1
+$EndComp
+Wire Wire Line
+	3300 9450 2850 9450
+Wire Wire Line
+	3300 9550 3100 9550
+Wire Wire Line
+	3100 9550 3100 9700
+$Comp
+L GND #PWR031
+U 1 1 5993D700
+P 3100 9700
+F 0 "#PWR031" H 3100 9450 50  0001 C CNN
+F 1 "GND" H 3100 9550 50  0000 C CNN
+F 2 "" H 3100 9700 50  0001 C CNN
+F 3 "" H 3100 9700 50  0001 C CNN
+	1    3100 9700
+	1    0    0    -1
+$EndComp
+Text Label 2850 9450 0    60   ~ 0
+L_OUT
 $EndSCHEMATC
